Commit message: Using newer nao model
source: https://raw.githubusercontent.com/stack-of-tasks/pinocchio-benchmarks/6bed73443d6cfdfcd732c171932bd905454dbc94/models/nao.urdf

File: examples/urdfreader/nao.urdf (robot description, URDF)
Before this commit: robot NaoH25V50, 79 links, 78 joints
Links:
- removed link CameraBottom_optical_frame
- removed link CameraTop_optical_frame
- removed link ChestButton_frame
- removed link HeadTouchFront_frame
- removed link HeadTouchMiddle_frame
- removed link HeadTouchRear_frame
- removed link ImuTorsoAccelerometer_frame
- removed link ImuTorsoGyrometer_frame
- removed link LAnklePitch
- removed link LFinger11_link
- removed link LFinger12_link
- removed link LFinger13_link
- removed link LFinger21_link
- removed link LFinger22_link
- removed link LFinger23_link
- removed link LFootBumperLeft_frame
- removed link LFootBumperRight_frame
- removed link LFsrFL_frame
- removed link LFsrFR_frame
- removed link LFsrRL_frame
- removed link LFsrRR_frame
- removed link LHandTouchBack_frame
- removed link LHandTouchLeft_frame
- removed link LHandTouchRight_frame
- removed link LInfraRed_frame
- removed link LSonar_frame
- removed link LThumb1_link
- removed link LThumb2_link
- removed link RAnklePitch
- removed link RFinger11_link
- removed link RFinger12_link
- removed link RFinger13_link
- removed link RFinger21_link
- removed link RFinger22_link
- removed link RFinger23_link
- removed link RFootBumperLeft_frame
- removed link RFootBumperRight_frame
- removed link RFsrFL_frame
- removed link RFsrFR_frame
- removed link RFsrRL_frame
- removed link RFsrRR_frame
- removed link RHandTouchBack_frame
- removed link RHandTouchLeft_frame
- removed link RHandTouchRight_frame
- removed link RInfraRed_frame
- removed link RSonar_frame
- removed link RThumb1_link
- removed link RThumb2_link
- removed link l_ankle
- removed link l_gripper
- removed link l_wrist
- removed link r_ankle
- removed link r_gripper
- removed link r_wrist
- removed link torso
- added link LAnkle, mass 0.13416; collision box size=0.078 0.028 0.058; visual mesh filename=package://nao_model/mesh/dae/LAnkle.dae
- added link LFeet, mass 0.16184; collision box size=0.161 0.088 0.064; visual mesh filename=package://nao_model/mesh/dae/LFeet.dae
- added link LFinger, mass 0; collision box size=0.04 0.04 0.04; visual mesh filename=package://nao_model/mesh/dae/LFinger.dae
- added link LHand, mass 0.18533; collision box size=0.084 0.068 0.063; visual mesh filename=package://nao_model/mesh/dae/LHand.dae
- added link RAnkle, mass 0.13415; collision box size=0.078 0.028 0.058; visual mesh filename=package://nao_model/mesh/dae/RAnkle.dae
- added link RFeet, mass 0.16171; collision box size=0.161 0.088 0.064; visual mesh filename=package://nao_model/mesh/dae/RFeet.dae
- added link RFinger, mass 0; collision box size=0.04 0.04 0.04; visual mesh filename=package://nao_model/mesh/dae/RFinger.dae
- added link RHand, mass 0.18533; collision box size=0.084 0.068 0.063; visual mesh filename=package://nao_model/mesh/dae/RHand.dae
- added link Torso, mass 1.04956; collision box size=0.111 0.192 0.23; visual mesh filename=package://nao_model/mesh/dae/Torso.dae
- link Head: geometry collision box size=0.119 0.133 0.116; visual mesh filename=package://nao_model/mesh/dae/Head.dae
- link LBicep: geometry collision box size=0.143 0.05 0.055; visual mesh filename=package://nao_model/mesh/dae/LBicep.dae
- link LForeArm: geometry collision box size=0.072 0.051 0.052; visual mesh filename=package://nao_model/mesh/dae/LForeArm.dae
- link LHip: mass 0.14053 -> 0.13053; geometry collision box size=0.076 0.028 0.049; visual mesh filename=package://nao_model/mesh/dae/LHip.dae
- link LPelvis: geometry collision box size=0.08 0.05 0.056; visual mesh filename=package://nao_model/mesh/dae/LPelvis.dae
- link LShoulder: mass 0.09304 -> 0.07504; geometry collision box size=0.061 0.057 0.082; visual mesh filename=package://nao_model/mesh/dae/LShoulder.dae
- link LThigh: geometry collision box size=0.095 0.089 0.143; visual mesh filename=package://nao_model/mesh/dae/LThigh.dae
- link LTibia: mass 0.30142 -> 0.29142; geometry collision box size=0.07 0.093 0.1; visual mesh filename=package://nao_model/mesh/dae/LTibia.dae
- link Neck: mass 0.07842 -> 0.06442; geometry 
- link RBicep: mass 0.15777 -> 0.15794; geometry collision box size=0.143 0.05 0.055; visual mesh filename=package://nao_model/mesh/dae/RBicep.dae
- link RForeArm: mass 0.07761 -> 0.07778; geometry collision box size=0.072 0.051 0.052; visual mesh filename=package://nao_model/mesh/dae/RForeArm.dae
- link RHip: mass 0.14053 -> 0.13053; geometry collision box size=0.076 0.028 0.049; visual mesh filename=package://nao_model/mesh/dae/RHip.dae
- link RPelvis: mass 0.06981 -> 0.07118; geometry collision box size=0.08 0.05 0.056; visual mesh filename=package://nao_model/mesh/dae/RPelvis.dae
- link RShoulder: mass 0.09304 -> 0.07504; geometry collision box size=0.061 0.057 0.082; visual mesh filename=package://nao_model/mesh/dae/RShoulder.dae
- link RThigh: mass 0.38968 -> 0.38976; geometry collision box size=0.095 0.089 0.143; visual mesh filename=package://nao_model/mesh/dae/RThigh.dae
- link RTibia: mass 0.30142 -> 0.29163; geometry collision box size=0.07 0.093 0.1; visual mesh filename=package://nao_model/mesh/dae/RTibia.dae
- link base_link: mass None -> 0.000001
Joints:
- removed joint Accelerometer_sensor_fixedjoint
- removed joint CameraBottom_optical_frame_fixedjoint
- removed joint CameraBottom_sensor_fixedjoint
- removed joint CameraTop_optical_frame_fixedjoint
- removed joint CameraTop_sensor_fixedjoint
- removed joint ChestBoard/Button_sensor_fixedjoint
- removed joint Gyrometer_sensor_fixedjoint
- removed joint Head/Touch/Front_sensor_fixedjoint
- removed joint Head/Touch/Middle_sensor_fixedjoint
- removed joint Head/Touch/Rear_sensor_fixedjoint
- removed joint InfraredL_sensor_fixedjoint
- removed joint InfraredR_sensor_fixedjoint
- removed joint LFinger11
- removed joint LFinger12
- removed joint LFinger13
- removed joint LFinger21
- removed joint LFinger22
- removed joint LFinger23
- removed joint LFoot/Bumper/Left_sensor_fixedjoint
- removed joint LFoot/Bumper/Right_sensor_fixedjoint
- removed joint LFoot/FSR/FrontLeft_sensor_fixedjoint
- removed joint LFoot/FSR/FrontRight_sensor_fixedjoint
- removed joint LFoot/FSR/RearLeft_sensor_fixedjoint
- removed joint LFoot/FSR/RearRight_sensor_fixedjoint
- removed joint LHand
- removed joint LHand/Touch/Back_sensor_fixedjoint
- removed joint LHand/Touch/Left_sensor_fixedjoint
- removed joint LHand/Touch/Right_sensor_fixedjoint
- removed joint LLeg_effector_fixedjoint
- removed joint LThumb1
- removed joint LThumb2
- removed joint RFinger11
- removed joint RFinger12
- removed joint RFinger13
- removed joint RFinger21
- removed joint RFinger22
- removed joint RFinger23
- removed joint RFoot/Bumper/Left_sensor_fixedjoint
- removed joint RFoot/Bumper/Right_sensor_fixedjoint
- removed joint RFoot/FSR/FrontLeft_sensor_fixedjoint
- removed joint RFoot/FSR/FrontRight_sensor_fixedjoint
- removed joint RFoot/FSR/RearLeft_sensor_fixedjoint
- removed joint RFoot/FSR/RearRight_sensor_fixedjoint
- removed joint RHand
- removed joint RHand/Touch/Back_sensor_fixedjoint
- removed joint RHand/Touch/Left_sensor_fixedjoint
- removed joint RHand/Touch/Right_sensor_fixedjoint
- removed joint RLeg_effector_fixedjoint
- removed joint RThumb1
- removed joint RThumb2
- removed joint Sonar/Left_sensor_fixedjoint
- removed joint Sonar/Right_sensor_fixedjoint
- removed joint base_link_fixedjoint
- added joint CameraBottom: type fixed, parent Head, child CameraBottom_frame, origin xyz=0.05071 0 0.01774 rpy=-2.263692 0 -1.57079632679
- added joint CameraTop: type fixed, parent Head, child CameraTop_frame, origin xyz=0.05871 0 0.06364 rpy=-1.59174 0 -1.57079632679
- added joint LGripper: type fixed, parent LHand, child LFinger, origin xyz=0 0 0
- added joint RGripper: type fixed, parent RHand, child RFinger, origin xyz=0 0 0
- added joint base_joint: type fixed, parent base_link, child Torso, origin xyz=0 0 0 rpy=0 0 0
- added joint l_sole_joint: type fixed, parent LFeet, child l_sole, origin xyz=0 0 0 rpy=0 0 0
- added joint r_sole_joint: type fixed, parent RFeet, child r_sole, origin xyz=0 0 0 rpy=0 0 0
- joint HeadPitch: axis 0 1.0 0 -> 0 1 0; limit lower=-0.671952 upper=0.514872 effort=1.532 velocity=7.19407 -> lower=-0.672 upper=0.5149 effort=100.0 velocity=5
- joint HeadYaw: axis 0 0 1.0 -> 0 0 1; limit lower=-2.08567 upper=2.08567 effort=1.547 velocity=8.26797 -> lower=-2.0857 upper=2.0857 effort=100.0 velocity=5; parent torso -> Torso
- joint LAnklePitch: axis 0 1.0 0 -> 0 1 0; child LAnklePitch -> LAnkle; limit lower=-1.18944 upper=0.922581 effort=3.023 velocity=6.40239 -> lower=-1.189516 upper=0.922747 effort=100.0 velocity=5; origin xyz=0 0 -0.1029 rpy=0 0 0 -> xyz=0 0 -0.10290 rpy=0 0 0
- joint LAnkleRoll: axis 1.0 0 0 -> 1 0 0; child l_ankle -> LFeet; limit lower=-0.397761 upper=0.768992 effort=3.348 velocity=4.16174 -> lower=-0.39788 upper=0.769001 effort=100.0 velocity=5; parent LAnklePitch -> LAnkle
- joint LElbowRoll: axis 0 0 1.0 -> 0 0 1; limit lower=-1.54462 upper=-0.0349066 effort=1.532 velocity=7.19407 -> lower=-1.5446 upper=-0.0349 effort=100.0 velocity=5
- joint LElbowYaw: axis 1.0 0 0 -> 1 0 0; limit lower=-2.08567 upper=2.08567 effort=1.547 velocity=8.26797 -> lower=-2.0857 upper=2.0857 effort=100.0 velocity=5
- joint LHipPitch: axis 0 1.0 0 -> 0 1 0; limit lower=-1.53589 upper=0.48398 effort=3.023 velocity=6.40239 -> lower=-1.773912 upper=0.48409 effort=100.0 velocity=5
- joint LHipRoll: axis 1.0 0 0 -> 1 0 0; limit lower=-0.379435 upper=0.79046 effort=3.348 velocity=4.16174 -> lower=-0.379472 upper=0.790477 effort=100.0 velocity=5
- joint LHipYawPitch: limit lower=-1.14529 upper=0.740718 effort=3.348 velocity=4.16174 -> lower=-1.145303 upper=0.74081 effort=100.0 velocity=5; parent torso -> Torso
- joint LKneePitch: axis 0 1.0 0 -> 0 1 0; limit lower=-0.0923279 upper=2.11255 effort=3.023 velocity=6.40239 -> lower=-0.092346 upper=2.112528 effort=100.0 velocity=5
- joint LShoulderPitch: axis 0 1.0 0 -> 0 1 0; limit lower=-2.08567 upper=2.08567 effort=1.329 velocity=8.26797 -> lower=-2.0857 upper=2.0857 effort=100.0 velocity=5; parent torso -> Torso
- joint LShoulderRoll: axis 0 0 1.0 -> 0 0 1; limit lower=-0.314159 upper=1.32645 effort=1.7835 velocity=7.19407 -> lower=-0.3142 upper=1.3265 effort=100.0 velocity=5
- joint LWristYaw: axis 1.0 0 0 -> 1 0 0; child l_wrist -> LHand; limit lower=-1.82387 upper=1.82387 effort=0.4075 velocity=24.6229 -> lower=-1.8238 upper=1.8238 effort=100.0 velocity=5
- joint RAnklePitch: axis 0 1.0 0 -> 0 1 0; child RAnklePitch -> RAnkle; limit lower=-1.1863 upper=0.932006 effort=3.0226 velocity=6.40239 -> lower=-1.186448 upper=0.932056 effort=100.0 velocity=5; origin xyz=0 0 -0.1029 rpy=0 0 0 -> xyz=0 0 -0.10290 rpy=0 0 0
- joint RAnkleRoll: axis 1.0 0 0 -> 1 0 0; child r_ankle -> RFeet; limit lower=-0.768992 upper=0.397761 effort=3.348 velocity=4.16174 -> lower=-0.785875 upper=0.388676 effort=100.0 velocity=5; parent RAnklePitch -> RAnkle
- joint RElbowRoll: axis 0 0 1.0 -> 0 0 1; limit lower=0.0349066 upper=1.54462 effort=1.532 velocity=7.19407 -> lower=0.0349 upper=1.5446 effort=100.0 velocity=5
- joint RElbowYaw: axis 1.0 0 0 -> 1 0 0; limit lower=-2.08567 upper=2.08567 effort=1.547 velocity=8.26797 -> lower=-2.0857 upper=2.0857 effort=100.0 velocity=5
- joint RHipPitch: axis 0 1.0 0 -> 0 1 0; limit lower=-1.53589 upper=0.48398 effort=3.0226 velocity=6.40239 -> lower=-1.772308 upper=0.485624 effort=100.0 velocity=5
- joint RHipRoll: axis 1.0 0 0 -> 1 0 0; limit lower=-0.79046 upper=0.379435 effort=3.348 velocity=4.16174 -> lower=-0.738321 upper=0.414754 effort=100.0 velocity=5
- joint RHipYawPitch: limit lower=-1.14529 upper=0.740718 effort=3.348 velocity=4.16174 -> lower=-1.145303 upper=0.74081 effort=100.0 velocity=5; mimic joint=LHipYawPitch multiplier=1.0 offset=0 -> (none); parent torso -> Torso
- joint RKneePitch: axis 0 1.0 0 -> 0 1 0; limit lower=-0.0923279 upper=2.11255 effort=3.0226 velocity=6.40239 -> lower=-0.103083 upper=2.120198 effort=100.0 velocity=5
- joint RShoulderPitch: axis 0 1.0 0 -> 0 1 0; limit lower=-2.08567 upper=2.08567 effort=1.329 velocity=8.26797 -> lower=-2.0857 upper=2.0857 effort=100.0 velocity=5; parent torso -> Torso
- joint RShoulderRoll: axis 0 0 1.0 -> 0 0 1; limit lower=-1.32645 upper=0.314159 effort=1.783 velocity=7.19407 -> lower=-1.3265 upper=0.3142 effort=100.0 velocity=5
- joint RWristYaw: axis 1.0 0 0 -> 1 0 0; child r_wrist -> RHand; limit lower=-1.82387 upper=1.82387 effort=0.4075 velocity=24.6229 -> lower=-1.8238 upper=1.8238 effort=100.0 velocity=5
- joint gaze_joint: origin xyz=0.05871 0 0.06364 rpy=0 0 0 -> xyz=0.0539 0 0.05
